File: ModuMixer X16/Controller board/DSP.kicad_sch (KiCad schematic)
At the start: 35 parts, among them U2 LM324, U6 TLV320AIC3100, U7 STM32F405RGTx, U9 AMS1117-1.8

Commit message: update idk
Parts:
- removed C55, C56: 47mF, Capacitor_SMD:C_0603_1608Metric, symbol Device:C
- removed unit 2 of U2
- added C41, C42: 47uF, Capacitor_SMD:C_0603_1608Metric, symbol Device:C
- added C68: 100nF, Capacitor_SMD:C_0603_1608Metric, symbol Device:C
- added C72: 100n, Capacitor_SMD:C_0603_1608Metric, symbol Device:C
- added Q3, Q4: MMBT2222A, Package_TO_SOT_SMD:SOT-23, symbol Transistor_BJT:MMBT2222A
- added R10, R11, R12, R9: 1k, Resistor_SMD:R_0603_1608Metric, symbol Device:R
- added R14, R15, R16, R17: 1k, symbol Device:R
- added TP13: SWCLK, TestPoint:TestPoint_Pad_D3.0mm, symbol Connector:TestPoint
- added TP14: SWIO, TestPoint:TestPoint_Pad_D3.0mm, symbol Connector:TestPoint
- added U11: LM358, Package_CSP:LFCSP-8_2x2mm_P0.5mm, symbol Amplifier_Operational:LM358
- added unit 3 of U5
- added unit 1 of U5
- added unit 2 of U5
- added unit 4 of U5
- added U9: 4016, Package_SO:SOIC-14_3.9x8.7mm_P1.27mm, symbol 4xxx:4016
- renumbered C58 to C38, C49 to C39, C50 to C40, C21 to C43, C59 to C44, C57 to C45, C60 to C46, C61 to C47, C39 to C48, C40 to C49, C62 to C50, C63 to C51, C43 to C52, C44 to C53, C64 to C54, C65 to C55, C41 to C56, C42 to C57, C66 to C58, C47 to C59, C48 to C60, C67 to C61, C68 to C62, C51 to C63, C52 to C64, C69 to C65, C53 to C66, C54 to C67, U2 to U5, U9 to U6, U6 to U7, U7 to U8
Connections:
- net 5V_MAIN: now also C68.1, Q3.3 (C), R12.2, U9.14 (VDD)
- net GND: now also C68.2, C72.2, Q4.2 (E), R10.1, U11.4 (V-), U5.12 (+), U5.3 (+), U9.7 (VSS)
- net HPL: now also C41.1
- net HPR: now also C42.1
- net MAIN_IN_R: now also U11.1, U11.2 (-)
- net MAIN_IN_R_P: now also U11.3 (+)
- net DSP_SPI_NSS: now reaches U8.20 (PA4)
- net DSP_SPI_SCK: now reaches U8.21 (PA5)
- net DSP_SPI_MISO: now reaches U8.22 (PA6)
- net DSP_SPI_MOSI: now reaches U8.23 (PA7)
- net DSP_SWIO: now reaches U8.46 (PA13)
- net DSP_SWIO: now also TP14.1
- net DSP_SWCLK: now reaches U8.49 (PA14)
- net DSP_SWCLK: now also TP13.1
- new net: R16.2, R17.1, U5.2 (-)
- new net: Q3.1 (B), R9.2
- new net: R14.2, R15.1, U5.13 (-)
- new net: Q4.1 (B), R11.2
- new net: C72.1, U11.8 (V+)
- new net CUE_CTRL: R9.1
- new net CUE_L: U9.3
- new net CUE_R: U9.10
- new net CUE_SEL: Q4.3 (C), R12.1, U9.12, U9.5
- new net HP_L: U5.8, U5.9 (-)
- new net HP_L_PRE: U5.10 (+), U9.2, U9.4
- new net HP_R: U5.6 (-), U5.7
- new net HP_R_PRE: U5.5 (+), U9.11, U9.9
- new net MAIN_L: U9.1
- new net MAIN_OUT_L_M: R15.2, U5.14
- new net MAIN_OUT_R_M: R17.2, U5.1
- new net MAIN_R: U9.8
- new net MAIN_SEL: Q3.2 (E), R10.2, R11.1, U9.13, U9.6
- new net OUT_L_PRE: C41.2, R14.1
- new net OUT_R_PRE: C42.2, R16.1
Other:
- moved on the sheet: C38, C39, C40, C43, C44, C45, C46, C47, U5E, U6, U7, U8

Commit message: idk testing github desktop
Parts:
- R14, R15, R16, R17: footprint (none) -> Resistor_SMD:R_0603_1608Metric
- U5: footprint (none) -> Package_SO:SOIC-14_3.9x8.7mm_P1.27mm
- U5: footprint Package_SO:TSSOP-14_4.4x5mm_P0.65mm -> Package_SO:SOIC-14_3.9x8.7mm_P1.27mm
Other:
- moved on the sheet: U11B
Changed lines of the file:
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@@
 	(symbol
 		(lib_id "Amplifier_Operational:LM358")
-		(at -25.4 114.3 0)
+		(at -12.7 137.16 0)
 		(unit 2)
 		(exclude_from_sim no)
@@
 		(fields_autoplaced yes)
 		(property "Reference" "U11"
-			(at -25.4 104.14 0)
+			(at -12.7 127 0)
 			(effects
 				(font
@@
 		)
 		(property "Value" "LM358"
-			(at -25.4 106.68 0)
+			(at -12.7 129.54 0)
 			(effects
 				(font
@@
 		)
 		(property "Footprint" "Package_CSP:LFCSP-8_2x2mm_P0.5mm"
-			(at -25.4 114.3 0)
+			(at -12.7 137.16 0)
 			(effects
 				(font
@@
 		)
 		(property "Datasheet" "http://www.ti.com/lit/ds/symlink/lm2904-n.pdf"
-			(at -25.4 114.3 0)
+			(at -12.7 137.16 0)
 			(effects
 				(font
@@
 		)
 		(property "Description" "Low-Power, Dual Operational Amplifiers, DIP-8/SOIC-8/TO-99-8"
-			(at -25.4 114.3 0)
+			(at -12.7 137.16 0)
 			(effects
 				(font
@@
 			)
 		)
-		(property "Footprint" ""
+		(property "Footprint" "Package_SO:SOIC-14_3.9x8.7mm_P1.27mm"
 			(at 86.36 111.76 0)
 			(effects
@@
 			)
 		)
-		(property "Footprint" ""
+		(property "Footprint" "Package_SO:SOIC-14_3.9x8.7mm_P1.27mm"
 			(at 125.73 114.3 0)
 			(effects
@@
 			)
 		)
-		(property "Footprint" ""
+		(property "Footprint" "Resistor_SMD:R_0603_1608Metric"
 			(at 127 130.048 90)
 			(effects
@@
 			)
 		)
-		(property "Footprint" ""
+		(property "Footprint" "Resistor_SMD:R_0603_1608Metric"
 			(at 115.57 121.158 90)
 			(effects
@@
 			)
 		)
-		(property "Footprint" ""
+		(property "Footprint" "Package_SO:SOIC-14_3.9x8.7mm_P1.27mm"
 			(at 86.36 92.71 0)
 			(effects
@@
 			)
 		)
-		(property "Footprint" ""
+		(property "Footprint" "Resistor_SMD:R_0603_1608Metric"
 			(at 115.57 97.028 90)
 			(effects
@@
 			)
 		)
-		(property "Footprint" ""
+		(property "Footprint" "Package_SO:SOIC-14_3.9x8.7mm_P1.27mm"
 			(at 125.73 90.17 0)
 			(effects
@@
 			)
 		)
-		(property "Footprint" "Package_SO:TSSOP-14_4.4x5mm_P0.65mm"
+		(property "Footprint" "Package_SO:SOIC-14_3.9x8.7mm_P1.27mm"
 			(at 33.02 107.95 0)
 			(effects
@@
 			)
 		)
-		(property "Footprint" ""
+		(property "Footprint" "Resistor_SMD:R_0603_1608Metric"
 			(at 127 105.918 90)
 			(effects
