File: ModuMixer X16/Controller board/PowerSupply.kicad_sch (KiCad schematic)
At the start: 44 parts, among them J6 Screw_Terminal_01x02, Q2 MMBT2222A, Q3 IRF9540N, SW26 SW_SPST, U3 LM317_TO-220, U4 LM317_TO-220, U5 LM317_TO-220

Commit message: MCU replacement finished
Parts:
- R10, R5, R6, R7, R8, R9: footprint Resistor_SMD:R_0201_0603Metric -> Resistor_SMD:R_0603_1608Metric
Connections:
- net +12V_MAIN is gone; now on net 12V_MAIN: C17.1, C18.1, C19.1, C20.1, C21.1, C22.1, C23.1, D1.1 (K), D2.1 (K), SW26.2 (B), U3.3 (VI), U4.3 (VI)
- net +12V_MOD is gone; now on net 12V_MOD: C33.1
- net +12V_IN renamed 12V_IN
Changed lines of the file:
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@@
 		)
 	)
-	(global_label "+12V_IN"
+	(global_label "12V_IN"
 		(shape bidirectional)
 		(at 110.49 21.59 180)
@@
 		)
 		(property "Intersheetrefs" "${INTERSHEET_REFS}"
-			(at 110.49 21.59 0)
+			(at 99.983 21.59 0)
 			(effects
 				(font
 					(size 1.27 1.27)
 				)
+				(justify right)
 				(hide yes)
 			)
 		)
 	)
-	(global_label "+12V_MAIN"
+	(global_label "12V_MAIN"
 		(shape bidirectional)
 		(at 35.56 48.26 180)
@@
 		)
 		(property "Intersheetrefs" "${INTERSHEET_REFS}"
-			(at 35.56 48.26 0)
+			(at 22.513 48.26 0)
 			(effects
 				(font
 					(size 1.27 1.27)
 				)
+				(justify right)
 				(hide yes)
 			)
 		)
 	)
-	(global_label "+12V_MAIN"
+	(global_label "12V_MAIN"
 		(shape bidirectional)
 		(at 35.56 85.09 180)
@@
 		)
 		(property "Intersheetrefs" "${INTERSHEET_REFS}"
-			(at 35.56 85.09 0)
+			(at 22.513 85.09 0)
 			(effects
 				(font
 					(size 1.27 1.27)
 				)
+				(justify right)
 				(hide yes)
 			)
@@
 		)
 	)
-	(global_label "+12V_IN"
+	(global_label "12V_IN"
 		(shape bidirectional)
 		(at 102.87 48.26 180)
@@
 		)
 		(property "Intersheetrefs" "${INTERSHEET_REFS}"
-			(at 102.87 48.26 0)
+			(at 92.363 48.26 0)
 			(effects
 				(font
 					(size 1.27 1.27)
 				)
+				(justify right)
 				(hide yes)
 			)
@@
 		)
 	)
-	(global_label "+12V_MAIN"
+	(global_label "12V_MAIN"
 		(shape bidirectional)
 		(at 87.63 21.59 0)
@@
 		)
 		(property "Intersheetrefs" "${INTERSHEET_REFS}"
-			(at 87.63 21.59 0)
+			(at 100.677 21.59 0)
 			(effects
 				(font
 					(size 1.27 1.27)
 				)
+				(justify left)
 				(hide yes)
 			)
@@
 		)
 		(property "Intersheetrefs" "${INTERSHEET_REFS}"
-			(at 195.58 46.99 0)
+			(at 208.627 46.99 0)
 			(effects
 				(font
 					(size 1.27 1.27)
 				)
+				(justify left)
 				(hide yes)
 			)
 		)
 	)
-	(global_label "+12V_MAIN"
+	(global_label "12V_MAIN"
 		(shape bidirectional)
 		(at 59.69 16.51 0)
@@
 		)
 		(property "Intersheetrefs" "${INTERSHEET_REFS}"
-			(at 59.69 16.51 0)
+			(at 72.737 16.51 0)
 			(effects
 				(font
 					(size 1.27 1.27)
 				)
+				(justify left)
 				(hide yes)
 			)
@@
 		)
 	)
-	(global_label "+12V_MOD"
+	(global_label "12V_MOD"
 		(shape bidirectional)
 		(at 213.36 48.26 0)
@@
 		)
 		(property "Intersheetrefs" "${INTERSHEET_REFS}"
-			(at 213.36 48.26 0)
+			(at 225.9836 48.26 0)
 			(effects
 				(font
 					(size 1.27 1.27)
 				)
+				(justify left)
 				(hide yes)
 			)
@@
 		)
 	)
-	(global_label "+12V_IN"
+	(global_label "12V_IN"
 		(shape bidirectional)
 		(at 77.47 21.59 180)
@@
 		)
 		(property "Intersheetrefs" "${INTERSHEET_REFS}"
-			(at 77.47 21.59 0)
+			(at 66.963 21.59 0)
 			(effects
 				(font
 					(size 1.27 1.27)
 				)
+				(justify right)
 				(hide yes)
 			)
@@
 			)
 		)
-		(property "Footprint" "Resistor_SMD:R_0201_0603Metric"
+		(property "Footprint" "Resistor_SMD:R_0603_1608Metric"
 			(at 58.928 97.79 90)
 			(effects
@@
 			)
 		)
-		(property "Footprint" "Resistor_SMD:R_0201_0603Metric"
+		(property "Footprint" "Resistor_SMD:R_0603_1608Metric"
 			(at 58.928 60.96 90)
 			(effects
@@
 			)
 		)
-		(property "Footprint" "Resistor_SMD:R_0201_0603Metric"
+		(property "Footprint" "Resistor_SMD:R_0603_1608Metric"
 			(at 69.342 52.07 90)
 			(effects
@@
 			)
 		)
-		(property "Footprint" "Resistor_SMD:R_0201_0603Metric"
+		(property "Footprint" "Resistor_SMD:R_0603_1608Metric"
 			(at 126.238 60.96 90)
 			(effects
@@
 			)
 		)
-		(property "Footprint" "Resistor_SMD:R_0201_0603Metric"
+		(property "Footprint" "Resistor_SMD:R_0603_1608Metric"
 			(at 136.652 52.07 90)
 			(effects
@@
 			)
 		)
-		(property "Footprint" "Resistor_SMD:R_0201_0603Metric"
+		(property "Footprint" "Resistor_SMD:R_0603_1608Metric"
 			(at 69.342 88.9 90)
 			(effects
